Commit message: Added derivatives

File: urdf_models/puma/puma.urdf (robot description, URDF)
Before this commit: robot Puma, 7 links, 6 joints
Links:
- added link end-effector-frame, mass 0.39
Joints:
- added joint wrist-roll3: type fixed, parent end-effector, child end-effector-frame, origin xyz=0.0 0.0 0.0 rpy=0.0 0.0 1.5707
