Commit message: added muscle jacobian derivative

File: examples/09-muscle/human.urdf (robot description, URDF)
Before this commit: robot human, 40 links, 39 joints
Links:
- link left_foot: geometry visual mesh filename=foot_l_1f.obj; visual mesh filename=toes_l_1f.obj
- link pelvis: mass 50.0 -> 20.0
- link right_foot: geometry visual mesh filename=foot_r_1f.obj; visual mesh filename=toes_r_1f.obj
Joints:
- joint left_ankle_pitch: limit lower=-0.65 upper=0.65 effort=100 velocity=10 -> lower=-0.65 upper=0.65 effort=200 velocity=10
- joint left_ankle_roll: limit lower=-0.65 upper=0.65 effort=100 velocity=10 -> lower=-0.65 upper=0.65 effort=200 velocity=10
- joint left_elbow_pitch: limit lower=-2.4 upper=-0.6 effort=100 velocity=10 -> lower=-2.4 upper=0 effort=200 velocity=10
- joint left_hip_pitch: limit lower=-0.4 upper=2.3 effort=100 velocity=10 -> lower=-2.3 upper=2.3 effort=200 velocity=10
- joint left_hip_roll: limit lower=-0.4 upper=0.4 effort=100 velocity=10 -> lower=-0.4 upper=0.4 effort=200 velocity=10
- joint left_hip_yaw: limit lower=-0.4 upper=2.3 effort=100 velocity=10 -> lower=-0.4 upper=2.3 effort=200 velocity=10
- joint left_knee_pitch: limit lower=-0.6 upper=2.5 effort=100 velocity=10 -> lower=0 upper=2.5 effort=200 velocity=10
- joint left_shoulder_pitch: limit lower=-1.8 upper=1.2 effort=100 velocity=10 -> lower=-1.8 upper=1.2 effort=200 velocity=10
- joint left_shoulder_roll: limit lower=-0.79 upper=0 effort=100 velocity=10 -> lower=-0.79 upper=0 effort=200 velocity=10
- joint left_shoulder_yaw: limit lower=-1.3 upper=0.2 effort=100 velocity=10 -> lower=-1.3 upper=0.2 effort=200 velocity=10
- joint left_toes_yaw: limit lower=-0.65 upper=0.65 effort=100 velocity=10 -> lower=-0.65 upper=0.65 effort=200 velocity=10
- joint left_wrist_pitch: limit lower=-0.9 upper=1.1 effort=100 velocity=10 -> lower=-0.9 upper=1.1 effort=200 velocity=10
- joint left_wrist_roll: limit lower=-0.9 upper=1.1 effort=100 velocity=10 -> lower=-0.9 upper=1.1 effort=200 velocity=10
- joint left_wrist_yaw: limit lower=-0.9 upper=1.1 effort=100 velocity=10 -> lower=-0.9 upper=1.1 effort=200 velocity=10
- joint neck_pitch: limit lower=-0.4 upper=0.79 effort=100 velocity=10 -> lower=-0.4 upper=0.79 effort=200 velocity=10
- joint neck_yaw: limit lower=-1.7 upper=1.7 effort=100 velocity=10 -> lower=-1.7 upper=1.7 effort=200 velocity=10
- joint right_ankle_pitch: limit lower=-0.65 upper=0.65 effort=100 velocity=10 -> lower=-0.65 upper=0.65 effort=200 velocity=10
- joint right_ankle_roll: limit lower=-0.65 upper=0.65 effort=100 velocity=10 -> lower=-0.65 upper=0.65 effort=200 velocity=10
- joint right_elbow_pitch: limit lower=-2.4 upper=-0.6 effort=100 velocity=10 -> lower=-2.4 upper=0 effort=200 velocity=10
- joint right_hip_pitch: limit lower=-2.3 upper=0.4 effort=100 velocity=10 -> lower=-2.3 upper=2.3 effort=200 velocity=10
- joint right_hip_roll: limit lower=-0.4 upper=0.4 effort=100 velocity=10 -> lower=-0.4 upper=0.4 effort=200 velocity=10
- joint right_hip_yaw: limit lower=-0.4 upper=0.4 effort=100 velocity=10 -> lower=-0.4 upper=0.4 effort=200 velocity=10
- joint right_knee_pitch: limit lower=0.6 upper=2.5 effort=100 velocity=10 -> lower=0 upper=2.5 effort=200 velocity=10
- joint right_shoulder_pitch: limit lower=-1.8 upper=1.2 effort=100 velocity=10 -> lower=-1.8 upper=1.2 effort=200 velocity=10
- joint right_shoulder_roll: limit lower=-0.79 upper=0 effort=100 velocity=10 -> lower=-0.79 upper=0 effort=200 velocity=10
- joint right_shoulder_yaw: limit lower=-1.3 upper=0.2 effort=100 velocity=10 -> lower=-1.3 upper=0.2 effort=200 velocity=10
- joint right_toes_yaw: limit lower=-0.65 upper=0.65 effort=100 velocity=10 -> lower=-0.65 upper=0.65 effort=200 velocity=10
- joint right_wrist_pitch: limit lower=-0.9 upper=1.1 effort=100 velocity=10 -> lower=-0.9 upper=1.1 effort=200 velocity=10
- joint right_wrist_roll: limit lower=-0.9 upper=1.1 effort=100 velocity=10 -> lower=-0.9 upper=1.1 effort=200 velocity=10
- joint right_wrist_yaw: limit lower=-0.9 upper=1.1 effort=100 velocity=10 -> lower=-0.9 upper=1.1 effort=200 velocity=10
- joint root_rot_x: limit lower=-100 upper=100 effort=39 velocity=1.3963 -> lower=-100 upper=100 effort=1000 velocity=1.3963
- joint root_rot_y: limit lower=-100 upper=100 effort=39 velocity=1.3963 -> lower=-100 upper=100 effort=1000 velocity=1.3963
- joint root_rot_z: limit lower=-100 upper=100 effort=39 velocity=1.3963 -> lower=-100 upper=100 effort=1000 velocity=1.3963
- joint root_trans_x: limit lower=-100 upper=100 effort=39 velocity=1.3963 -> lower=-100 upper=100 effort=1000 velocity=1.3963
- joint root_trans_y: limit lower=-100 upper=100 effort=39 velocity=1.3963 -> lower=-100 upper=100 effort=1000 velocity=1.3963
- joint root_trans_z: limit lower=-100 upper=100 effort=39 velocity=1.3963 -> lower=-100 upper=100 effort=1000 velocity=1.3963
- joint waist_pitch: limit lower=-0.83 upper=0.83 effort=100 velocity=10 -> lower=-0.83 upper=0.83 effort=200 velocity=10
- joint waist_roll: limit lower=-1.1 upper=1.1 effort=100 velocity=10 -> lower=-1.1 upper=1.1 effort=200 velocity=10
- joint waist_yaw: limit lower=-0.83 upper=0.83 effort=100 velocity=10 -> lower=-0.83 upper=0.83 effort=200 velocity=10

Commit message: revised muscle jacobian matrix and derivative to match opensim

File: examples/09-muscle/human.urdf (robot description, URDF)
Before this commit: robot humanoid_clean, 40 links, 39 joints
Joints:
- joint neck_pitch: limit lower=-0.4 upper=0.79 effort=200 velocity=10 -> (none); type revolute -> fixed
- joint neck_yaw: limit lower=-1.7 upper=1.7 effort=200 velocity=10 -> (none); type revolute -> fixed
